File: UC-50-001.kicad_sch (KiCad schematic)
At the start: 0 parts

Commit message: commence PIA
Other:
- sheet PIA - ports clavier, crayon optique et LEP renamed I48–MC6821P - ports clavier, crayon optique et LEP
Changed lines of the file:
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@@
     (stroke (width 0.1524) (type solid) (color 0 0 0 0))
     (fill (color 0 0 0 0.0000))
-    (property "Sheet name" "PIA - ports clavier, crayon optique et LEP" (id 0) (at 30.48 87.9234 0)
+    (property "Sheet name" "I48–MC6821P - ports clavier, crayon optique et LEP" (id 0) (at 30.48 87.9234 0)
       (effects (font (size 1.8 1.8)) (justify left bottom))
     )
@@
       (reference "#PWR?") (unit 1) (value "+5V") (footprint "")
     )
+    (path "/b7e71b61-5858-491f-a12d-087d8cf2d648/505ba418-ffce-4763-b84e-18836353024d"
+      (reference "#PWR?") (unit 1) (value "GND") (footprint "")
+    )
+    (path "/b7e71b61-5858-491f-a12d-087d8cf2d648/56378a1d-8ca6-405e-82ce-5f206f3fa204"
+      (reference "#PWR?") (unit 1) (value "GND") (footprint "")
+    )
     (path "/afd59d07-bfd6-4bc9-8176-e0ddec1872a1/601e7756-9222-41ed-b96b-8651f8dceb01"
       (reference "#PWR?") (unit 1) (value "GND") (footprint "")
@@
       (reference "#PWR?") (unit 1) (value "GND") (footprint "")
     )
+    (path "/b7e71b61-5858-491f-a12d-087d8cf2d648/8bd665a3-d2bc-4eb9-ab07-d1b073552cd5"
+      (reference "#PWR?") (unit 1) (value "+5V") (footprint "")
+    )
     (path "/f465a4b1-7c3c-40cc-9e66-ff9f17003d42/91b9ef3b-7eda-43c9-9d9b-33dfe0701bf3"
       (reference "#PWR?") (unit 1) (value "+5V") (footprint "")
@@
       (reference "#PWR?") (unit 1) (value "+5V") (footprint "")
     )
+    (path "/b7e71b61-5858-491f-a12d-087d8cf2d648/a90f36dc-a633-4fa2-8d93-d71e6e97e77f"
+      (reference "#PWR?") (unit 1) (value "+5V") (footprint "")
+    )
     (path "/706ec47c-3d4a-4bde-bb8b-c4f8dcc96c45/b62f804f-0408-4609-af13-f9d6c2a09a8a"
       (reference "#PWR?") (unit 1) (value "GND") (footprint "")
     )
+    (path "/b7e71b61-5858-491f-a12d-087d8cf2d648/b68ac7f1-e39a-4351-983f-a83005cfb447"
+      (reference "#PWR?") (unit 1) (value "GND") (footprint "")
+    )
     (path "/b7e71b61-5858-491f-a12d-087d8cf2d648/b95ce775-5d6b-4e74-ba16-0b8e6240d3e2"
       (reference "#PWR?") (unit 1) (value "+5V") (footprint "")
@@
       (reference "#PWR?") (unit 1) (value "+5V") (footprint "")
     )
+    (path "/b7e71b61-5858-491f-a12d-087d8cf2d648/cc2f772d-66f5-4ef2-bf72-bf4cabe8468e"
+      (reference "#PWR?") (unit 1) (value "GND") (footprint "")
+    )
     (path "/afd59d07-bfd6-4bc9-8176-e0ddec1872a1/d396128e-0019-4b81-b8de-65492819bfe3"
+      (reference "#PWR?") (unit 1) (value "GND") (footprint "")
+    )
+    (path "/b7e71b61-5858-491f-a12d-087d8cf2d648/e0fb4996-14ac-4391-982b-b8f6ac20cf31"
       (reference "#PWR?") (unit 1) (value "GND") (footprint "")
     )
@@
       (reference "C01") (unit 1) (value "100uF") (footprint "")
     )
+    (path "/b7e71b61-5858-491f-a12d-087d8cf2d648/36dce4c7-2705-4bcb-b676-3fb13d1e9187"
+      (reference "C7") (unit 1) (value "220nF") (footprint "")
+    )
+    (path "/b7e71b61-5858-491f-a12d-087d8cf2d648/e3e2211a-0ffd-4c3c-a583-5bbc586c5560"
+      (reference "C08") (unit 1) (value "220nF") (footprint "")
+    )
+    (path "/b7e71b61-5858-491f-a12d-087d8cf2d648/68a94170-63f4-456f-9e5a-d0abdde61225"
+      (reference "C09") (unit 1) (value "220nF") (footprint "")
+    )
+    (path "/b7e71b61-5858-491f-a12d-087d8cf2d648/905132d1-d645-461b-8a0a-367aa1adfb7f"
+      (reference "C10") (unit 1) (value "220nF") (footprint "")
+    )
+    (path "/b7e71b61-5858-491f-a12d-087d8cf2d648/1358d05d-bbca-4178-806c-95be186bd553"
+      (reference "C11") (unit 1) (value "220nF") (footprint "")
+    )
+    (path "/b7e71b61-5858-491f-a12d-087d8cf2d648/3bb57e2e-345e-4062-9f4d-e50f564cb519"
+      (reference "C12") (unit 1) (value "6.8nF") (footprint "")
+    )
+    (path "/b7e71b61-5858-491f-a12d-087d8cf2d648/f5257546-8197-49be-a359-f5c83042be18"
+      (reference "C16") (unit 1) (value "220nF") (footprint "")
+    )
+    (path "/b7e71b61-5858-491f-a12d-087d8cf2d648/98bf4bcf-04c1-4978-a311-bbe1510cbb4b"
+      (reference "C18") (unit 1) (value "10nF") (footprint "")
+    )
+    (path "/b7e71b61-5858-491f-a12d-087d8cf2d648/55193726-317e-40af-a41a-426c4f2665c3"
+      (reference "C19") (unit 1) (value "220nF") (footprint "")
+    )
+    (path "/b7e71b61-5858-491f-a12d-087d8cf2d648/9dae772a-3c96-437b-a8f7-ba96ede29d3c"
+      (reference "C20") (unit 1) (value "4.7uF") (footprint "")
+    )
     (path "/afd59d07-bfd6-4bc9-8176-e0ddec1872a1/9f60c894-1671-4e7a-aa00-77d68a3255ef"
       (reference "C21") (unit 1) (value "47nF") (footprint "")
@@
       (reference "C37") (unit 1) (value "47nF") (footprint "")
     )
+    (path "/b7e71b61-5858-491f-a12d-087d8cf2d648/7b50f0b0-2f53-40ee-88db-486e413d7af1"
+      (reference "C39") (unit 1) (value "47nF") (footprint "")
+    )
+    (path "/b7e71b61-5858-491f-a12d-087d8cf2d648/14ae1964-1d5a-41bc-ade1-66894bb82355"
+      (reference "C61") (unit 1) (value "6.8nF") (footprint "")
+    )
     (path "/b7e71b61-5858-491f-a12d-087d8cf2d648/9aaeccc0-c91f-4e78-ae85-1d4c16274d09"
       (reference "C?") (unit 1) (value "100uF") (footprint "")
@@
       (reference "I48") (unit 1) (value "PERIPHERAL_INTERFACE_ADAPTER_PHY") (footprint "Package_DIP:DIP-40_W15.24mm_LongPads")
     )
+    (path "/b7e71b61-5858-491f-a12d-087d8cf2d648/5999c531-4211-49b6-9884-4f174640d57f"
+      (reference "PM01") (unit 1) (value "DIN-5 Port LEP") (footprint "")
+    )
+    (path "/b7e71b61-5858-491f-a12d-087d8cf2d648/eb2b926a-99e6-4ebd-a9fa-857e8a3af559"
+      (reference "PM02") (unit 1) (value "DIN-5 Port Crayon optique") (footprint "")
+    )
     (path "/afd59d07-bfd6-4bc9-8176-e0ddec1872a1/79fa233e-a3b4-4a75-b36c-997bfb744c5f"
       (reference "R07") (unit 1) (value "680") (footprint "")
@@
       (reference "R33") (unit 1) (value "1K") (footprint "")
     )
+    (path "/b7e71b61-5858-491f-a12d-087d8cf2d648/f6934876-7f17-4d7e-bec9-35b9ebc47134"
+      (reference "R48") (unit 1) (value "1K") (footprint "")
+    )
+    (path "/b7e71b61-5858-491f-a12d-087d8cf2d648/a0cf2de4-4c25-42d7-9828-38c186d8d2d1"
+      (reference "R49") (unit 1) (value "1K") (footprint "")
+    )
+    (path "/b7e71b61-5858-491f-a12d-087d8cf2d648/a5f31b07-fa1d-494d-9dd6-2d023f919ef4"
+      (reference "R50") (unit 1) (value "1K") (footprint "")
+    )
+    (path "/b7e71b61-5858-491f-a12d-087d8cf2d648/88c5af05-cf53-48b7-af2c-4ffca662a157"
+      (reference "R51") (unit 1) (value "1K") (footprint "")
+    )
+    (path "/b7e71b61-5858-491f-a12d-087d8cf2d648/d389d950-bd1a-4513-b93e-fc155116e0f5"
+      (reference "R53") (unit 1) (value "33K") (footprint "")
+    )
+    (path "/b7e71b61-5858-491f-a12d-087d8cf2d648/14b66a4b-39b6-4a9b-8811-93f667907db8"
+      (reference "R56") (unit 1) (value "1K") (footprint "")
+    )
+    (path "/b7e71b61-5858-491f-a12d-087d8cf2d648/60af3131-3a88-4ebb-8604-c67ace5851d0"
+      (reference "R71") (unit 1) (value "100K") (footprint "")
+    )
+    (path "/b7e71b61-5858-491f-a12d-087d8cf2d648/74dd670a-3af9-4c07-aa2f-9ff33e25004f"
+      (reference "R72") (unit 1) (value "39K") (footprint "")
+    )
+    (path "/b7e71b61-5858-491f-a12d-087d8cf2d648/6f98cf7a-57f2-4f6e-9447-f98e33107a55"
+      (reference "R75") (unit 1) (value "15K") (footprint "")
+    )
+    (path "/b7e71b61-5858-491f-a12d-087d8cf2d648/97905e19-bd3d-4b37-9af1-07f470383640"
+      (reference "R76") (unit 1) (value "3K9") (footprint "")
+    )
+    (path "/b7e71b61-5858-491f-a12d-087d8cf2d648/16eb3702-915f-4f9c-9b46-548b3890cf9e"
+      (reference "R77") (unit 1) (value "1K") (footprint "")
+    )
     (path "/b7e71b61-5858-491f-a12d-087d8cf2d648/495713af-606d-4ff5-8146-89c3d23d953c"
       (reference "R?") (unit 1) (value "1K") (footprint "")
@@
       (reference "S01") (unit 1) (value "Initial Prog.") (footprint "")
     )
+    (path "/b7e71b61-5858-491f-a12d-087d8cf2d648/cb3eda70-4f82-436a-8212-b27f1a0704c3"
+      (reference "T11") (unit 1) (value "BC 547 B") (footprint "")
+    )
     (path "/3b9df46e-3592-4470-9765-1c36c3c4b1c2/1425be50-4ffe-4685-9900-caf49649b930"
