File: subsheet_103.kicad_sch (KiCad schematic)
At the start: 35 parts, among them T11 BC 547 B

Commit message: RAM : temporairement fini
Connections:
- net LIGHT PEN INT: now reaches I48.40 (CA1)
- net OPTIC PEN 1 renamed LIGHT PEN 1
- net OPTIC PEN 4 renamed LIGHT PEN 4
Changed lines of the file:
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@@
+    (stroke (width 0) (type default) (color 0 0 0 0))
+  )
+  (wire (pts (xy 168.91 59.69) (xy 180.34 59.69))
     (stroke (width 0) (type default) (color 0 0 0 0))
   )
@@
     (effects (font (size 1.27 1.27)) (justify left bottom))
   )
-  (text "de I09-11" (at 168.91 59.69 0)
-    (effects (font (size 1.27 1.27)) (justify left bottom))
+  (text "de I09-11" (at 180.34 59.69 180)
+    (effects (font (size 1.27 1.27)) (justify right bottom))
   )
   (label "1Y1" (at 36.83 144.78 0)
@@
     )
   )
-  (global_label "OPTIC PEN 4" (shape output) (at 48.26 59.69 0) (fields_autoplaced)
-    (effects (font (size 1.27 1.27)) (justify left))
-    (property "Intersheet References" "${INTERSHEET_REFS}" (id 0) (at 63.0102 59.7694 0)
+  (global_label "LIGHT PEN 4" (shape output) (at 48.26 59.69 0) (fields_autoplaced)
+    (effects (font (size 1.27 1.27)) (justify left))
+    (property "Intersheet References" "${INTERSHEET_REFS}" (id 0) (at 62.7683 59.6106 0)
+      (effects (font (size 1.27 1.27)) (justify left) hide)
+    )
+  )
+  (global_label "LIGHT PEN INT" (shape input) (at 180.34 59.69 0) (fields_autoplaced)
+    (effects (font (size 1.27 1.27)) (justify left))
+    (property "Intersheet References" "${INTERSHEET_REFS}" (id 0) (at 196.5417 59.6106 0)
       (effects (font (size 1.27 1.27)) (justify left) hide)
     )
@@
     )
   )
-  (global_label "OPTIC PEN 1" (shape output) (at 48.26 36.83 0) (fields_autoplaced)
-    (effects (font (size 1.27 1.27)) (justify left))
-    (property "Intersheet References" "${INTERSHEET_REFS}" (id 0) (at 63.0102 36.7506 0)
-      (effects (font (size 1.27 1.27)) (justify left) hide)
-    )
+  (global_label "LIGHT PEN 1" (shape output) (at 48.26 36.83 0) (fields_autoplaced)
+    (effects (font (size 1.27 1.27)) (justify left))
+    (property "Intersheet References" "${INTERSHEET_REFS}" (id 0) (at 62.7683 36.7506 0)
+      (effects (font (size 1.27 1.27)) (justify left) hide)
+    )
