File: subsheet_107.kicad_sch (KiCad schematic)
At the start: 0 parts

Commit message: commence le circuit d'alimentation
Parts:
- added C54: 10uF, symbol Device:C_Polarized_Small
- added C? (x3): 47nF, symbol Device:C_Small
- added C? (x2): 100uF, symbol Device:C_Polarized_Small
- added C?: 10nF, symbol Device:C_Small
- added D07: BYW98-100, symbol Device:D_Small
- added D?: 1N4148, symbol Device:D_Small
- added I55: LM311N Comparateur différentiel, Package_DIP:DIP-8_W7.62mm_LongPads, symbol lm311:DIFFERENTIAL_COMPARATORS_PHY
- added L02: 350uH, symbol Device:L_Small
- added PM03: Prise alimentation, symbol Connector:Jack-DC
- added R78, R?: 1K, symbol Device:R_Small
- added R81: 330, symbol Device:R_Small
- added R?: 3K3, symbol Device:R_Small
- added T12: BDX54, symbol Device:Q_PNP_EBC
- added U?: L78L05_TO92, Package_TO_SOT_THT:TO-92_Inline, symbol Regulator_Linear:L78L05_TO92
Connections:
- new net: C54.1, R81.1, U?.1 (VO)
- new net: I55.3 (IN-), R81.2
- new net +15V: PM03.2, U?.3 (VI)
- new net +5V: C?.1, C?.2
- new net GND: C54.2, C?.1, C?.2, I55.4 (VCC-), PM03.1, U?.2 (GND)
Other:
- note added: "Masse au centre"
- title: (none) -> Conversion du Thomson MO5 — Unité centrale

Commit message: remise au propre
Parts:
- removed C? (x3): 47nF, symbol Device:C_Small
- removed C?: 10nF, symbol Device:C_Small
- removed C?: 100uF, symbol Device:C_Polarized_Small
- removed D?: 1N4148, symbol Device:D_Small
- removed R?: 3K3, symbol Device:R_Small
- removed R?: 1K, symbol Device:R_Small
- added C55: 470uF, symbol Device:C_Polarized_Small
- added C56: 1000uF, symbol Device:C_Polarized_Small
- added L03: 15uH, symbol Device:L_Small
- added R79: 15K, symbol Device:R_Small
- added R80: 47K, symbol Device:R_Small
- added R83: 330, symbol Device:R_Small
- gave numbers to parts that had none: 1
Connections:
- net +15V: now also C?.1, I55.8 (VCC+), R78.1, T12.1 (E)
- net +5V: now also C56.1, L03.2
- net GND: now also C?.2, D07.2 (A), C55.2, C56.2
- net at I55.2 (IN+): now also C55.1, R80.2, R83.1
- net at I55.7 (COL_OUT): now also R79.2, R80.1
- net at D07.1 (K): now also L02.1, T12.3 (C)
- net at R78.2: now also T12.2 (B), R79.1
- net at L02.2: now also L03.1, R83.2
- no-connect marks 0 -> 3
Other:
- note added: "14.5V"
- note added: "17.4V"
- note added: "5V"
- title: Conversion du Thomson MO5 — Unité centrale -> Conversion du Thomson MO5 — Unité centrale v1
- moved on the sheet: C54, C?, D07, I54, I55, L02, PM03, R78, R81, T12

Commit message: horloges : stylo optique
Other:
- note added: "14,5V"
- note added: "17,4V"
- note removed: "17.4V"
Changed lines of the file:
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@@
     (effects (font (size 1.27 1.27)) (justify left bottom))
   )
-  (text "14.5V" (at 106.68 39.37 0)
+  (text "14,5V" (at 106.68 39.37 0)
     (effects (font (size 1.27 1.27)) (justify left bottom))
   )
-  (text "17.4V" (at 90.17 41.91 0)
+  (text "17,4V" (at 90.17 41.91 0)
     (effects (font (size 1.27 1.27)) (justify left bottom))
   )

Commit message: Point de test 1
Parts:
- added ZW01: TestPoint, symbol Connector:TestPoint
Connections:
- net +15V: now also ZW01.1
Other:
- moved on the sheet: PM03
Changed lines of the file:
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@@
     (comment 4 "Reference : POP5001 501994-01")
   )
-  (junction (at 43.18 96.52) (diameter 0) (color 0 0 0 0)
+  (junction (at 60.96 101.6) (diameter 0) (color 0 0 0 0)
+  )
+  (junction (at 41.91 96.52) (diameter 0) (color 0 0 0 0)
   )
   (junction (at 137.16 59.69) (diameter 0) (color 0 0 0 0)
@@
   (junction (at 121.92 59.69) (diameter 0) (color 0 0 0 0)
   )
-  (junction (at 52.07 101.6) (diameter 0) (color 0 0 0 0)
-  )
-  (junction (at 57.15 101.6) (diameter 0) (color 0 0 0 0)
+  (junction (at 50.8 101.6) (diameter 0) (color 0 0 0 0)
+  )
+  (junction (at 55.88 101.6) (diameter 0) (color 0 0 0 0)
   )
   (junction (at 91.44 46.99) (diameter 0) (color 0 0 0 0)
@@
     (stroke (width 0) (type default) (color 0 0 0 0))
   )
-  (wire (pts (xy 38.1 96.52) (xy 43.18 96.52))
+  (wire (pts (xy 36.83 96.52) (xy 41.91 96.52))
     (stroke (width 0) (type default) (color 0 0 0 0))
   )
@@
     (stroke (width 0) (type default) (color 0 0 0 0))
   )
+  (wire (pts (xy 60.96 101.6) (xy 66.04 101.6))
+    (stroke (width 0) (type default) (color 0 0 0 0))
+  )
   (wire (pts (xy 71.12 46.99) (xy 76.2 46.99))
     (stroke (width 0) (type default) (color 0 0 0 0))
@@
     (stroke (width 0) (type default) (color 0 0 0 0))
   )
-  (wire (pts (xy 38.1 101.6) (xy 52.07 101.6))
+  (wire (pts (xy 36.83 101.6) (xy 50.8 101.6))
     (stroke (width 0) (type default) (color 0 0 0 0))
   )
@@
     (stroke (width 0) (type default) (color 0 0 0 0))
   )
-  (wire (pts (xy 43.18 96.52) (xy 48.26 96.52))
+  (wire (pts (xy 41.91 96.52) (xy 46.99 96.52))
     (stroke (width 0) (type default) (color 0 0 0 0))
   )
@@
     (stroke (width 0) (type default) (color 0 0 0 0))
   )
-  (wire (pts (xy 52.07 101.6) (xy 57.15 101.6))
+  (wire (pts (xy 50.8 101.6) (xy 55.88 101.6))
     (stroke (width 0) (type default) (color 0 0 0 0))
   )
@@
     (stroke (width 0) (type default) (color 0 0 0 0))
   )
-  (wire (pts (xy 57.15 101.6) (xy 66.04 101.6))
+  (wire (pts (xy 55.88 101.6) (xy 60.96 101.6))
     (stroke (width 0) (type default) (color 0 0 0 0))
   )
@@
     (stroke (width 0) (type default) (color 0 0 0 0))
   )
-  (text "Masse au centre" (at 22.86 109.22 0)
+  (text "Masse au centre" (at 21.59 109.22 0)
     (effects (font (size 1.27 1.27)) (justify left bottom))
   )
@@
     (pin "2")
   )
+  (symbol (lib_id "Connector:TestPoint") (at 60.96 101.6 180) (unit 1)
+    (in_bom yes) (on_board yes)
+    (property "Reference" "ZW01" (id 0) (at 60.96 106.68 0))
+    (property "Value" "TestPoint" (id 1) (at 60.96 108.712 0))
+    (property "Footprint" "" (id 2) (at 55.88 101.6 0)
+      (effects (font (size 1.27 1.27)) hide)
+    )
+    (property "Datasheet" "~" (id 3) (at 55.88 101.6 0)
+      (effects (font (size 1.27 1.27)) hide)
+    )
+    (pin "1")
+  )
   (symbol (lib_id "Device:C_Polarized_Small") (at 153.67 53.34 0) (unit 1)
     (in_bom yes) (on_board yes)
@@
     (pin "2")
   )
-  (symbol (lib_id "power-custom:+18V") (at 57.15 101.6 0) (unit 1)
-    (in_bom yes) (on_board yes)
-    (property "Reference" "#PWR?" (id 0) (at 57.15 105.41 0)
-      (effects (font (size 1.27 1.27)) hide)
-    )
-    (property "Value" "+18V" (id 1) (at 57.15 98.044 0))
-    (property "Footprint" "" (id 2) (at 57.15 101.6 0)
-      (effects (font (size 1.27 1.27)) hide)
-    )
-    (property "Datasheet" "" (id 3) (at 57.15 101.6 0)
+  (symbol (lib_id "power-custom:+18V") (at 55.88 101.6 0) (unit 1)
+    (in_bom yes) (on_board yes)
+    (property "Reference" "#PWR?" (id 0) (at 55.88 105.41 0)
+      (effects (font (size 1.27 1.27)) hide)
+    )
+    (property "Value" "+18V" (id 1) (at 55.88 98.044 0))
+    (property "Footprint" "" (id 2) (at 55.88 101.6 0)
+      (effects (font (size 1.27 1.27)) hide)
+    )
+    (property "Datasheet" "" (id 3) (at 55.88 101.6 0)
       (effects (font (size 1.27 1.27)) hide)
     )
@@
     (pin "2")
   )
-  (symbol (lib_id "power:GND") (at 48.26 96.52 0) (unit 1)
-    (in_bom yes) (on_board yes)
-    (property "Reference" "#PWR?" (id 0) (at 48.26 102.87 0)
-      (effects (font (size 1.27 1.27)) hide)
-    )
-    (property "Value" "GND" (id 1) (at 46.99 99.06 0)
+  (symbol (lib_id "power:GND") (at 46.99 96.52 0) (unit 1)
+    (in_bom yes) (on_board yes)
+    (property "Reference" "#PWR?" (id 0) (at 46.99 102.87 0)
+      (effects (font (size 1.27 1.27)) hide)
+    )
+    (property "Value" "GND" (id 1) (at 45.72 99.06 0)
       (effects (font (size 1.27 1.27)) (justify right))
     )
-    (property "Footprint" "" (id 2) (at 48.26 96.52 0)
-      (effects (font (size 1.27 1.27)) hide)
-    )
-    (property "Datasheet" "" (id 3) (at 48.26 96.52 0)
-      (effects (font (size 1.27 1.27)) hide)
-    )
-    (pin "1")
-  )
-  (symbol (lib_id "Connector:Jack-DC") (at 30.48 99.06 0) (unit 1)
-    (in_bom yes) (on_board yes)
-    (property "Reference" "PM03" (id 0) (at 30.48 93.726 0))
-    (property "Value" "Prise alimentation" (id 1) (at 30.48 104.14 0))
-    (property "Footprint" "" (id 2) (at 31.75 100.076 0)
-      (effects (font (size 1.27 1.27)) hide)
-    )
-    (property "Datasheet" "~" (id 3) (at 31.75 100.076 0)
+    (property "Footprint" "" (id 2) (at 46.99 96.52 0)
+      (effects (font (size 1.27 1.27)) hide)
+    )
+    (property "Datasheet" "" (id 3) (at 46.99 96.52 0)
+      (effects (font (size 1.27 1.27)) hide)
+    )
+    (pin "1")
+  )
+  (symbol (lib_id "Connector:Jack-DC") (at 29.21 99.06 0) (unit 1)
+    (in_bom yes) (on_board yes)
+    (property "Reference" "PM03" (id 0) (at 29.21 93.726 0))
+    (property "Value" "Prise alimentation" (id 1) (at 29.21 104.14 0))
+    (property "Footprint" "" (id 2) (at 30.48 100.076 0)
+      (effects (font (size 1.27 1.27)) hide)
+    )
+    (property "Datasheet" "~" (id 3) (at 30.48 100.076 0)
       (effects (font (size 1.27 1.27)) hide)
     )
@@
     (pin "1")
   )
-  (symbol (lib_id "power:PWR_FLAG") (at 43.18 96.52 0) (unit 1)
-    (in_bom yes) (on_board yes)
-    (property "Reference" "#FLG?" (id 0) (at 43.18 94.615 0)
-      (effects (font (size 1.27 1.27)) hide)
-    )
-    (property "Value" "PWR_FLAG" (id 1) (at 43.18 92.71 0))
-    (property "Footprint" "" (id 2) (at 43.18 96.52 0)
-      (effects (font (size 1.27 1.27)) hide)
-    )
-    (property "Datasheet" "~" (id 3) (at 43.18 96.52 0)
+  (symbol (lib_id "power:PWR_FLAG") (at 41.91 96.52 0) (unit 1)
+    (in_bom yes) (on_board yes)
+    (property "Reference" "#FLG?" (id 0) (at 41.91 94.615 0)
+      (effects (font (size 1.27 1.27)) hide)
+    )
+    (property "Value" "PWR_FLAG" (id 1) (at 41.91 92.71 0))
+    (property "Footprint" "" (id 2) (at 41.91 96.52 0)
+      (effects (font (size 1.27 1.27)) hide)
+    )
+    (property "Datasheet" "~" (id 3) (at 41.91 96.52 0)
       (effects (font (size 1.27 1.27)) hide)
     )
@@
     (pin "1")
   )
-  (symbol (lib_id "power:PWR_FLAG") (at 52.07 101.6 180) (unit 1)
-    (in_bom yes) (on_board yes)
-    (property "Reference" "#FLG?" (id 0) (at 52.07 103.505 0)
-      (effects (font (size 1.27 1.27)) hide)
-    )
-    (property "Value" "PWR_FLAG" (id 1) (at 52.07 105.41 0))
-    (property "Footprint" "" (id 2) (at 52.07 101.6 0)
-      (effects (font (size 1.27 1.27)) hide)
-    )
-    (property "Datasheet" "~" (id 3) (at 52.07 101.6 0)
-      (effects (font (size 1.27 1.27)) hide)
-    )
+  (symbol (lib_id "power:PWR_FLAG") (at 50.8 101.6 180) (unit 1)
+    (in_bom yes) (on_board yes)
+    (property "Reference" "#FLG?" (id 0) (at 50.8 103.505 0)
+      (effects (font (size 1.27 1.27)) hide)
+    )
+    (property "Value" "PWR_FLAG" (id 1) (at 50.8 105.41 0))
+    (property "Footprint" "" (id 2) (at 50.8 101.6 0)
+      (effects (font (size 1.27 1.27)) hide)
+    )
+    (property "Datasheet" "~" (id 3) (at 50.8 101.6 0)
+      (effects (font (size 1.27 1.27)) hide)
+    )
