File: subsheet_105.kicad_sch (KiCad schematic)
At the start: 39 parts, among them T01 BC547B, T02 BC547B, T03 BC547B

Commit message: start association symbols-footprints
Parts:
- C22, C26, C30, C32, C36, C59: footprint (none) -> commons-passives_THT:Passive_THT_capacitor_mlcc_W2.54mm_L5.08mm
- D04, D05, D06: footprint (none) -> commons-passives_THT:Passive_THT_diode_W2.54mm_L12.70mm
- R01, R02, R03, R04, R05, R06, R14, R15, R16, R17, R18, R19, R20, R21, R22, R23, R24, R25, R26, R27, R28: footprint (none) -> commons-passives_THT:Passive_THT_resistor_EU_W2.54mm_L12.70mm
Changed lines of the file:
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@@
       (effects (font (size 1.27 1.27)) (justify right))
     )
-    (property "Footprint" "" (id 2) (at 55.88 195.58 0)
+    (property "Footprint" "commons-passives_THT:Passive_THT_resistor_EU_W2.54mm_L12.70mm" (id 2) (at 55.88 195.58 0)
       (effects (font (size 1.27 1.27)) hide)
     )
@@
       (effects (font (size 1.27 1.27)) (justify left))
     )
-    (property "Footprint" "" (id 2) (at 62.23 224.79 0)
+    (property "Footprint" "commons-passives_THT:Passive_THT_resistor_EU_W2.54mm_L12.70mm" (id 2) (at 62.23 224.79 0)
       (effects (font (size 1.27 1.27)) hide)
     )
@@
       (effects (font (size 1.27 1.27)) (justify right))
     )
-    (property "Footprint" "" (id 2) (at 104.14 246.38 0)
+    (property "Footprint" "commons-passives_THT:Passive_THT_resistor_EU_W2.54mm_L12.70mm" (id 2) (at 104.14 246.38 0)
       (effects (font (size 1.27 1.27)) hide)
     )
@@
       (effects (font (size 1.27 1.27)) (justify right))
     )
-    (property "Footprint" "" (id 2) (at 104.14 182.88 0)
+    (property "Footprint" "commons-passives_THT:Passive_THT_resistor_EU_W2.54mm_L12.70mm" (id 2) (at 104.14 182.88 0)
       (effects (font (size 1.27 1.27)) hide)
     )
@@
       (effects (font (size 1.27 1.27)) (justify right))
     )
-    (property "Footprint" "" (id 2) (at 83.82 121.92 0)
+    (property "Footprint" "commons-passives_THT:Passive_THT_capacitor_mlcc_W2.54mm_L5.08mm" (id 2) (at 83.82 121.92 0)
       (effects (font (size 1.27 1.27)) hide)
     )
@@
       (effects (font (size 1.27 1.27)) (justify left))
     )
-    (property "Footprint" "" (id 2) (at 101.6 215.9 90)
+    (property "Footprint" "commons-passives_THT:Passive_THT_diode_W2.54mm_L12.70mm" (id 2) (at 101.6 215.9 90)
       (effects (font (size 1.27 1.27)) hide)
     )
@@
       (effects (font (size 1.27 1.27)) (justify right))
     )
-    (property "Footprint" "" (id 2) (at 55.88 246.38 0)
+    (property "Footprint" "commons-passives_THT:Passive_THT_resistor_EU_W2.54mm_L12.70mm" (id 2) (at 55.88 246.38 0)
       (effects (font (size 1.27 1.27)) hide)
     )
@@
       (effects (font (size 1.27 1.27)) (justify right))
     )
-    (property "Footprint" "" (id 2) (at 161.29 208.28 0)
+    (property "Footprint" "commons-passives_THT:Passive_THT_capacitor_mlcc_W2.54mm_L5.08mm" (id 2) (at 161.29 208.28 0)
       (effects (font (size 1.27 1.27)) hide)
     )
@@
       (effects (font (size 1.27 1.27)) (justify right))
     )
-    (property "Footprint" "" (id 2) (at 104.14 233.68 0)
+    (property "Footprint" "commons-passives_THT:Passive_THT_resistor_EU_W2.54mm_L12.70mm" (id 2) (at 104.14 233.68 0)
       (effects (font (size 1.27 1.27)) hide)
     )
@@
       (effects (font (size 1.27 1.27)) (justify right))
     )
-    (property "Footprint" "" (id 2) (at 86.36 213.36 0)
+    (property "Footprint" "commons-passives_THT:Passive_THT_resistor_EU_W2.54mm_L12.70mm" (id 2) (at 86.36 213.36 0)
       (effects (font (size 1.27 1.27)) hide)
     )
@@
       (effects (font (size 1.27 1.27)) (justify left))
     )
-    (property "Footprint" "" (id 2) (at 101.6 190.5 90)
+    (property "Footprint" "commons-passives_THT:Passive_THT_diode_W2.54mm_L12.70mm" (id 2) (at 101.6 190.5 90)
       (effects (font (size 1.27 1.27)) hide)
     )
@@
       (effects (font (size 1.27 1.27)) (justify left))
     )
-    (property "Footprint" "" (id 2) (at 62.23 199.39 0)
+    (property "Footprint" "commons-passives_THT:Passive_THT_resistor_EU_W2.54mm_L12.70mm" (id 2) (at 62.23 199.39 0)
       (effects (font (size 1.27 1.27)) hide)
     )
@@
       (effects (font (size 1.27 1.27)) (justify right))
     )
-    (property "Footprint" "" (id 2) (at 170.18 63.5 0)
+    (property "Footprint" "commons-passives_THT:Passive_THT_capacitor_mlcc_W2.54mm_L5.08mm" (id 2) (at 170.18 63.5 0)
       (effects (font (size 1.27 1.27)) hide)
     )
@@
       (effects (font (size 1.27 1.27)) (justify right))
     )
-    (property "Footprint" "" (id 2) (at 55.88 220.98 0)
+    (property "Footprint" "commons-passives_THT:Passive_THT_resistor_EU_W2.54mm_L12.70mm" (id 2) (at 55.88 220.98 0)
       (effects (font (size 1.27 1.27)) hide)
     )
@@
       (effects (font (size 1.27 1.27)) (justify left))
     )
-    (property "Footprint" "" (id 2) (at 101.6 241.3 90)
+    (property "Footprint" "commons-passives_THT:Passive_THT_diode_W2.54mm_L12.70mm" (id 2) (at 101.6 241.3 90)
       (effects (font (size 1.27 1.27)) hide)
     )
@@
       (effects (font (size 1.27 1.27)) (justify right))
     )
-    (property "Footprint" "" (id 2) (at 104.14 195.58 0)
+    (property "Footprint" "commons-passives_THT:Passive_THT_resistor_EU_W2.54mm_L12.70mm" (id 2) (at 104.14 195.58 0)
       (effects (font (size 1.27 1.27)) hide)
     )
@@
       (effects (font (size 1.27 1.27)) (justify right))
     )
-    (property "Footprint" "" (id 2) (at 101.6 219.71 0)
+    (property "Footprint" "commons-passives_THT:Passive_THT_capacitor_mlcc_W2.54mm_L5.08mm" (id 2) (at 101.6 219.71 0)
       (effects (font (size 1.27 1.27)) hide)
     )
@@
       (effects (font (size 1.27 1.27)) (justify right))
     )
-    (property "Footprint" "" (id 2) (at 86.36 190.5 0)
+    (property "Footprint" "commons-passives_THT:Passive_THT_resistor_EU_W2.54mm_L12.70mm" (id 2) (at 86.36 190.5 0)
       (effects (font (size 1.27 1.27)) hide)
     )
@@
       (effects (font (size 1.27 1.27)) (justify left))
     )
-    (property "Footprint" "" (id 2) (at 76.2 194.31 0)
+    (property "Footprint" "commons-passives_THT:Passive_THT_resistor_EU_W2.54mm_L12.70mm" (id 2) (at 76.2 194.31 0)
       (effects (font (size 1.27 1.27)) hide)
     )
@@
       (effects (font (size 1.27 1.27)) (justify right))
     )
-    (property "Footprint" "" (id 2) (at 104.14 208.28 0)
+    (property "Footprint" "commons-passives_THT:Passive_THT_resistor_EU_W2.54mm_L12.70mm" (id 2) (at 104.14 208.28 0)
       (effects (font (size 1.27 1.27)) hide)
     )
@@
       (effects (font (size 1.27 1.27)) (justify right))
     )
-    (property "Footprint" "" (id 2) (at 86.36 187.96 0)
+    (property "Footprint" "commons-passives_THT:Passive_THT_resistor_EU_W2.54mm_L12.70mm" (id 2) (at 86.36 187.96 0)
       (effects (font (size 1.27 1.27)) hide)
     )
@@
       (effects (font (size 1.27 1.27)) (justify right))
     )
-    (property "Footprint" "" (id 2) (at 87.63 63.5 0)
+    (property "Footprint" "commons-passives_THT:Passive_THT_capacitor_mlcc_W2.54mm_L5.08mm" (id 2) (at 87.63 63.5 0)
       (effects (font (size 1.27 1.27)) hide)
     )
@@
       (effects (font (size 1.27 1.27)) (justify right))
     )
-    (property "Footprint" "" (id 2) (at 166.37 121.92 0)
+    (property "Footprint" "commons-passives_THT:Passive_THT_capacitor_mlcc_W2.54mm_L5.08mm" (id 2) (at 166.37 121.92 0)
       (effects (font (size 1.27 1.27)) hide)
     )
@@
       (effects (font (size 1.27 1.27)) (justify left))
     )
-    (property "Footprint" "" (id 2) (at 76.2 245.11 0)
+    (property "Footprint" "commons-passives_THT:Passive_THT_resistor_EU_W2.54mm_L12.70mm" (id 2) (at 76.2 245.11 0)
       (effects (font (size 1.27 1.27)) hide)
     )
@@
       (effects (font (size 1.27 1.27)) (justify right))
     )
-    (property "Footprint" "" (id 2) (at 86.36 241.3 0)
+    (property "Footprint" "commons-passives_THT:Passive_THT_resistor_EU_W2.54mm_L12.70mm" (id 2) (at 86.36 241.3 0)
       (effects (font (size 1.27 1.27)) hide)
     )
@@
       (effects (font (size 1.27 1.27)) (justify right))
     )
-    (property "Footprint" "" (id 2) (at 104.14 224.79 0)
+    (property "Footprint" "commons-passives_THT:Passive_THT_resistor_EU_W2.54mm_L12.70mm" (id 2) (at 104.14 224.79 0)
       (effects (font (size 1.27 1.27)) hide)
     )
@@
       (effects (font (size 1.27 1.27)) (justify left))
     )
-    (property "Footprint" "" (id 2) (at 76.2 219.71 0)
+    (property "Footprint" "commons-passives_THT:Passive_THT_resistor_EU_W2.54mm_L12.70mm" (id 2) (at 76.2 219.71 0)
       (effects (font (size 1.27 1.27)) hide)
     )
@@
       (effects (font (size 1.27 1.27)) (justify right))
     )
-    (property "Footprint" "" (id 2) (at 86.36 215.9 0)
+    (property "Footprint" "commons-passives_THT:Passive_THT_resistor_EU_W2.54mm_L12.70mm" (id 2) (at 86.36 215.9 0)
       (effects (font (size 1.27 1.27)) hide)
     )
@@
       (effects (font (size 1.27 1.27)) (justify right))
     )
-    (property "Footprint" "" (id 2) (at 86.36 238.76 0)
+    (property "Footprint" "commons-passives_THT:Passive_THT_resistor_EU_W2.54mm_L12.70mm" (id 2) (at 86.36 238.76 0)
       (effects (font (size 1.27 1.27)) hide)
     )
@@
       (effects (font (size 1.27 1.27)) (justify left))
     )
-    (property "Footprint" "" (id 2) (at 62.23 250.19 0)
-      (effects (font (size 1.27 1.27)) hide)
-    )
+    (property "Footprint" "commons-passives_THT:Passive_THT_resistor_EU_W2.54mm_L12.70mm" (id 2) (at 62.23 250.19 0)
+      (effects (font (size 1.27 1.27)) hide)
+    )

Commit message: continue footprints-symbols association
Parts:
- T01, T02, T03: footprint (none) -> Package_TO_SOT_THT:TO-92_Inline_Wide
Changed lines of the file:
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@@
       (effects (font (size 1.27 1.27)) (justify left))
     )
-    (property "Footprint" "" (id 2) (at 64.77 238.76 0)
+    (property "Footprint" "Package_TO_SOT_THT:TO-92_Inline_Wide" (id 2) (at 64.77 238.76 0)
       (effects (font (size 1.27 1.27)) hide)
     )
@@
       (effects (font (size 1.27 1.27)) (justify left))
     )
-    (property "Footprint" "" (id 2) (at 64.77 187.96 0)
+    (property "Footprint" "Package_TO_SOT_THT:TO-92_Inline_Wide" (id 2) (at 64.77 187.96 0)
       (effects (font (size 1.27 1.27)) hide)
     )
@@
       (effects (font (size 1.27 1.27)) (justify left))
     )
-    (property "Footprint" "" (id 2) (at 64.77 213.36 0)
-      (effects (font (size 1.27 1.27)) hide)
-    )
+    (property "Footprint" "Package_TO_SOT_THT:TO-92_Inline_Wide" (id 2) (at 64.77 213.36 0)
+      (effects (font (size 1.27 1.27)) hide)
+    )
