File: subsheet_104.kicad_sch (KiCad schematic)
At the start: 6 parts

Commit message: start association symbols-footprints
Parts:
- C25: footprint (none) -> commons-passives_THT:Passive_THT_capacitor_mlcc_W2.54mm_L5.08mm
Changed lines of the file:
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@@
       (effects (font (size 1.27 1.27)) (justify right))
     )
-    (property "Footprint" "" (id 2) (at 113.03 40.64 0)
+    (property "Footprint" "commons-passives_THT:Passive_THT_capacitor_mlcc_W2.54mm_L5.08mm" (id 2) (at 113.03 40.64 0)
       (effects (font (size 1.27 1.27)) hide)
     )

Commit message: continue footprints-symbols association
Parts:
- ZW02: footprint (none) -> Connector_PinHeader_2.54mm:PinHeader_1x01_P2.54mm_Vertical
Changed lines of the file:
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@@
     (property "Reference" "ZW02" (id 0) (at 73.66 186.182 0))
     (property "Value" "TestPoint" (id 1) (at 73.66 187.96 0))
-    (property "Footprint" "" (id 2) (at 78.74 193.04 0)
+    (property "Footprint" "Connector_PinHeader_2.54mm:PinHeader_1x01_P2.54mm_Vertical" (id 2) (at 78.74 193.04 0)
       (effects (font (size 1.27 1.27)) hide)
     )

Commit message: created cartridge footprint and associated with symbol in schematics
Parts:
- B06: footprint (none) -> thomson-moto-interconnect:cartridge_port_2x13_pcb_edge_pitch_100mils_row_pitch_200mils
Changed lines of the file:
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@@
     (property "Reference" "B06" (id 0) (at 101.6 111.76 0))
     (property "Value" "Port cartouche (rangée 'a' vers le sud)" (id 1) (at 101.6 152.4 0))
-    (property "Footprint" "" (id 2) (at 100.33 132.08 0)
+    (property "Footprint" "thomson-moto-interconnect:cartridge_port_2x13_pcb_edge_pitch_100mils_row_pitch_200mils" (id 2) (at 100.33 132.08 0)
       (effects (font (size 1.27 1.27)) hide)
     )

Commit message: associate extension ports with their footprints
Parts:
- B01: footprint (none) -> thomson-moto-interconnect:extension_port_1x19_backside_2mm_pad_width_2.54mm_pad_pitch
- B02: footprint (none) -> thomson-moto-interconnect:extension_port_1x19_topside_2mm_pad_width_2.54mm_pad_pitch
Changed lines of the file:
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@@
     (property "Reference" "B02" (id 0) (at 121.92 190.5 0))
     (property "Value" "Connecteur extension (dessus)" (id 1) (at 121.92 241.3 0))
-    (property "Footprint" "" (id 2) (at 121.92 215.9 0)
+    (property "Footprint" "thomson-moto-interconnect:extension_port_1x19_topside_2mm_pad_width_2.54mm_pad_pitch" (id 2) (at 121.92 215.9 0)
       (effects (font (size 1.27 1.27)) hide)
     )
@@
     (property "Reference" "B01" (id 0) (at 83.82 190.5 0))
     (property "Value" "Connecteur extension (dessous)" (id 1) (at 83.82 241.3 0))
-    (property "Footprint" "" (id 2) (at 83.82 215.9 0)
-      (effects (font (size 1.27 1.27)) hide)
-    )
+    (property "Footprint" "thomson-moto-interconnect:extension_port_1x19_backside_2mm_pad_width_2.54mm_pad_pitch" (id 2) (at 83.82 215.9 0)
+      (effects (font (size 1.27 1.27)) hide)
+    )
