File: subsheet_108.kicad_sch (KiCad schematic)
At the start: 16 parts

Commit message: pcb session 2024-03-24T08:04:18+01:00 -- routing, I20[12,13] to be left unwired
Connections:
- net GND: no longer I20.12 (4A), I20.13 (4B)
- no-connect marks 1 -> 3
Changed lines of the file:
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@@
   (junction (at 109.22 68.58) (diameter 0) (color 0 0 0 0)
   )
-  (junction (at 146.05 218.44) (diameter 0) (color 0 0 0 0)
-  )
   (junction (at 67.31 170.18) (diameter 0) (color 0 0 0 0)
   )
@@
   (junction (at 67.31 205.74) (diameter 0) (color 0 0 0 0)
   )
-  (junction (at 146.05 205.74) (diameter 0) (color 0 0 0 0)
-  )
   (junction (at 101.6 48.26) (diameter 0) (color 0 0 0 0)
   )
@@
   (junction (at 104.14 220.98) (diameter 0) (color 0 0 0 0)
   )
+  (no_connect (at 139.7 220.98))
+  (no_connect (at 139.7 218.44))
   (no_connect (at 139.7 223.52))
   (wire (pts (xy 100.33 228.6) (xy 106.68 228.6))
@@
     (stroke (width 0) (type default))
   )
-  (wire (pts (xy 146.05 220.98) (xy 146.05 218.44))
-    (stroke (width 0) (type default))
-  )
   (wire (pts (xy 63.5 220.98) (xy 68.58 220.98))
     (stroke (width 0) (type default))
@@
     (stroke (width 0) (type default))
   )
-  (wire (pts (xy 146.05 218.44) (xy 146.05 205.74))
-    (stroke (width 0) (type default))
-  )
   (wire (pts (xy 152.4 107.95) (xy 152.4 106.68))
     (stroke (width 0) (type default))
@@
     (stroke (width 0) (type default))
   )
-  (wire (pts (xy 139.7 220.98) (xy 146.05 220.98))
-    (stroke (width 0) (type default))
-  )
   (wire (pts (xy 93.98 58.42) (xy 101.6 58.42))
     (stroke (width 0) (type default))
@@
     (stroke (width 0) (type default))
   )
-  (wire (pts (xy 146.05 205.74) (xy 148.59 205.74))
+  (wire (pts (xy 140.97 205.74) (xy 148.59 205.74))
     (stroke (width 0) (type default))
   )
@@
     (stroke (width 0) (type default))
   )
-  (wire (pts (xy 139.7 218.44) (xy 146.05 218.44))
-    (stroke (width 0) (type default))
-  )
   (wire (pts (xy 38.1 71.12) (xy 60.96 71.12))
     (stroke (width 0) (type default))
@@
     (stroke (width 0) (type default))
   )
-  (wire (pts (xy 140.97 205.74) (xy 146.05 205.74))
-    (stroke (width 0) (type default))
-  )
