File: subsheet_109.kicad_sch (KiCad schematic)
At the start: 3 parts

Commit message: mentions of the motherboards revisions
Other:
- note added: "Les modules mémoire I100, I101 et I102 sont implantables uniquement sur les révisions POP 5007S et POP 5009S de la carte-mère."
Changed lines of the file:
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@@
     (rev "v2.0.0-alpha")
     (comment 1 "http://github.com/sporniket/kicad-conversions--thomson-mo5--v1")
-    (comment 3 "Gate Array EFCIS")
+    (comment 3 "Gate Array EFCIS EFG-J033-E / Matra-Harris MA4-Q1200 (POP 5007S, POP 5009S)")
+    (comment 4 "Références : POP 5003S, POP 5005S, POP 5007S, POP 5009S")
   )
   (wire (pts (xy 104.14 111.76) (xy 109.22 111.76))
@@
     (effects (font (size 1.27 1.27)) (justify right bottom))
   )
+  (text "Les modules mémoire I100, I101 et I102 sont implantables uniquement sur les révisions POP 5007S et POP 5009S de la carte-mère."
+    (at 41.91 34.29 0)
+    (effects (font (size 1.27 1.27)) (justify left bottom))
+  )
   (label "MA1" (at 104.14 106.68 0) (fields_autoplaced)
