File: UC-50-001.kicad_pcb (KiCad board)
At the start: 2 copper layers, 283 x 177.5 mm, 255 parts, among them J01 Jumper Wire, J02 Jumper Wire, J03 Jumper wire, J04 Jumper wire, J05 Jumper Wire, J07 Jumper wire, P01 1K, P02 ?, Q01 16MHz, T01 BC547B, T02 BC547B, T03 BC547B, T04 BC557B, T05 BC547B, T06 BC547B, T07 BC547B, T08 BC557B, T09 BC547B, T10 BC547B, T11 BC547B, T12 BDX54, T13 BC547B

Commit message: [pcb] area A.2, most of I40
Routing:
- net ADDR8: track 0.00 -> 375.2 mm, vias 0 -> 12
- net ADDR10: track 0.00 -> 303.2 mm, vias 0 -> 10
- net ADDR9: track 0.00 -> 207.8 mm, vias 0 -> 5
- net ADDR3: track 0.00 -> 206.1 mm, vias 0 -> 6
- net ADDR11: track 0.00 -> 117.6 mm, vias 0 -> 5
- net ADDR6: track 0.00 -> 96.2 mm, vias 0 -> 4
- net ADDR7: track 0.00 -> 93.2 mm, vias 0 -> 4
- net ADDR2: track 0.00 -> 71.0 mm, vias 0 -> 4
- net ~{A3}: track 0.00 -> 68.7 mm, vias 0 -> 2
- net ADDR12: track 265.7 -> 311.8 mm
- net ~{A4}: track 0.00 -> 26.2 mm, vias 0 -> 2
- net ~{A5}: track 0.00 -> 20.2 mm
- net Net-(I48-PA5): track 438.6 -> 450.2 mm
- net E: track 74.9 -> 81.1 mm
- net GND: track 1945.9 -> 1951.3 mm
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